File: Lowduino/LowduinoPTH_v2.sch (EAGLE design)
At the start: 23 parts, among them Q1 32.768kHz, U1 ATMEGA328P_PDIP

Commit message: Moved 1V8 voltage regulators from DensityAltitude.lbr to 1V8.lbr More layout work for various high input voltage regulators A bit more work on LowduinoPTH_v2
Parts:
- CN1: device adafruit:JST_2PIN-THM -> SparkFun-Connectors:M02JST-PTH-VERT
- U2: value (none) -> MCP1700-1802E/TO; device SparkFun-PowerIC:V_REG_78XXTO-92_UNTESTED -> 1V8:MCP1700-1802E/TO
Connections:
- net 1.8V: now also U2.VOUT; no longer U2.OUT
- net N$7: now also U2.VIN; no longer U2.IN
Other:
- moved on the sheet: C12, C13, CN1
Changed lines of the file:
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@@
 <part name="C2" library="SparkFun-Passives" deviceset="CAP" device="PTH1" value="0.1uF"/>
 <part name="SUPPLY5" library="SparkFun-Aesthetics" deviceset="1.8V" device=""/>
-<part name="U2" library="SparkFun-PowerIC" deviceset="V_REG_78XX" device="TO-92_UNTESTED"/>
 <part name="F1" library="SparkFun-PowerIC" deviceset="PTC" device="PTH"/>
 <part name="C3" library="SparkFun-Capacitors" deviceset="CAP" device="PTH"/>
@@
 <part name="JP2" library="SparkFun-Connectors" deviceset="ARDUINO_SERIAL_PROGRAM" device="PTH"/>
 <part name="JP5" library="SparkFun-Connectors" deviceset="M06" device="NO_SILK_FEMALE_PTH"/>
-<part name="CN1" library="adafruit" deviceset="JST_2PIN" device="-THM"/>
+<part name="CN1" library="SparkFun-Connectors" deviceset="M02" device="JST-PTH-VERT"/>
 <part name="JP6" library="SparkFun-Connectors" deviceset="M06" device="NO_SILK_FEMALE_PTH"/>
 <part name="S1" library="Lowduino" deviceset="MJTP_6MM" device=""/>
 <part name="JP4" library="SparkFun-Connectors" deviceset="M05" device="NO_SILK"/>
 <part name="JP7" library="SparkFun-Connectors" deviceset="M04" device="NO_SILK_ALL_ROUND"/>
+<part name="U2" library="1V8" deviceset="MCP1700" device="TO" technology="-1802E/"/>
 </parts>
 <sheets>
@@
 <instance part="JP1" gate="A" x="101.6" y="144.78"/>
 <instance part="GND3" gate="1" x="114.3" y="134.62"/>
-<instance part="GND4" gate="1" x="83.82" y="76.2"/>
+<instance part="GND4" gate="1" x="137.16" y="76.2"/>
 <instance part="C10" gate="G$1" x="60.96" y="88.9"/>
 <instance part="C11" gate="G$1" x="71.12" y="91.44"/>
-<instance part="C12" gate="G$1" x="96.52" y="91.44"/>
-<instance part="C13" gate="G$1" x="106.68" y="88.9"/>
+<instance part="C12" gate="G$1" x="149.86" y="91.44"/>
+<instance part="C13" gate="G$1" x="160.02" y="88.9"/>
 <instance part="D1" gate="G$1" x="53.34" y="96.52"/>
 <instance part="U1" gate="G$1" x="68.58" y="40.64"/>
@@
 <instance part="GND5" gate="1" x="17.78" y="2.54"/>
 <instance part="L1" gate="G$1" x="27.94" y="60.96" rot="R90"/>
-<instance part="SUPPLY2" gate="G$1" x="99.06" y="104.14"/>
+<instance part="SUPPLY2" gate="G$1" x="152.4" y="104.14"/>
 <instance part="SUPPLY3" gate="G$1" x="17.78" y="132.08"/>
 <instance part="GND6" gate="1" x="30.48" y="111.76"/>
 <instance part="C2" gate="G$1" x="30.48" y="121.92"/>
 <instance part="SUPPLY5" gate="G$1" x="114.3" y="152.4"/>
-<instance part="U2" gate="G$1" x="83.82" y="96.52"/>
 <instance part="F1" gate="G$1" x="38.1" y="96.52"/>
 <instance part="C3" gate="G$1" x="17.78" y="30.48"/>
@@
 <instance part="JP2" gate="G$1" x="121.92" y="116.84" rot="R180"/>
 <instance part="JP5" gate="G$1" x="139.7" y="60.96" rot="R180"/>
-<instance part="CN1" gate="G$1" x="20.32" y="96.52" rot="R180"/>
+<instance part="CN1" gate="G$1" x="20.32" y="93.98"/>
 <instance part="JP6" gate="G$1" x="139.7" y="12.7" rot="R180"/>
 <instance part="S1" gate="G$1" x="66.04" y="116.84" rot="R90"/>
 <instance part="JP4" gate="G$1" x="142.24" y="38.1" rot="R180"/>
 <instance part="JP7" gate="G$1" x="152.4" y="27.94" rot="R180"/>
+<instance part="U2" gate="A" x="93.98" y="93.98"/>
 </instances>
 <busses>
@@
 <segment>
 <pinref part="GND4" gate="1" pin="GND"/>
-<wire x1="83.82" y1="88.9" x2="83.82" y2="83.82" width="0.1524" layer="91"/>
+<wire x1="137.16" y1="88.9" x2="137.16" y2="83.82" width="0.1524" layer="91"/>
 <pinref part="C11" gate="G$1" pin="-"/>
-<wire x1="83.82" y1="83.82" x2="83.82" y2="78.74" width="0.1524" layer="91"/>
+<wire x1="137.16" y1="83.82" x2="137.16" y2="78.74" width="0.1524" layer="91"/>
 <wire x1="71.12" y1="86.36" x2="71.12" y2="83.82" width="0.1524" layer="91"/>
-<wire x1="71.12" y1="83.82" x2="83.82" y2="83.82" width="0.1524" layer="91"/>
-<junction x="83.82" y="83.82"/>
+<wire x1="71.12" y1="83.82" x2="93.98" y2="83.82" width="0.1524" layer="91"/>
+<junction x="137.16" y="83.82"/>
 <pinref part="C10" gate="G$1" pin="2"/>
+<wire x1="93.98" y1="83.82" x2="137.16" y2="83.82" width="0.1524" layer="91"/>
 <wire x1="60.96" y1="86.36" x2="60.96" y2="83.82" width="0.1524" layer="91"/>
 <wire x1="60.96" y1="83.82" x2="71.12" y2="83.82" width="0.1524" layer="91"/>
 <junction x="71.12" y="83.82"/>
 <pinref part="C12" gate="G$1" pin="-"/>
-<wire x1="83.82" y1="83.82" x2="96.52" y2="83.82" width="0.1524" layer="91"/>
-<wire x1="96.52" y1="83.82" x2="96.52" y2="86.36" width="0.1524" layer="91"/>
+<wire x1="137.16" y1="83.82" x2="149.86" y2="83.82" width="0.1524" layer="91"/>
+<wire x1="149.86" y1="83.82" x2="149.86" y2="86.36" width="0.1524" layer="91"/>
 <pinref part="C13" gate="G$1" pin="2"/>
-<wire x1="96.52" y1="83.82" x2="106.68" y2="83.82" width="0.1524" layer="91"/>
-<wire x1="106.68" y1="83.82" x2="106.68" y2="86.36" width="0.1524" layer="91"/>
-<junction x="96.52" y="83.82"/>
+<wire x1="149.86" y1="83.82" x2="160.02" y2="83.82" width="0.1524" layer="91"/>
+<wire x1="160.02" y1="83.82" x2="160.02" y2="86.36" width="0.1524" layer="91"/>
+<junction x="149.86" y="83.82"/>
 <wire x1="27.94" y1="83.82" x2="60.96" y2="83.82" width="0.1524" layer="91"/>
 <junction x="60.96" y="83.82"/>
-<wire x1="22.86" y1="93.98" x2="27.94" y2="93.98" width="0.1524" layer="91"/>
 <wire x1="27.94" y1="93.98" x2="27.94" y2="83.82" width="0.1524" layer="91"/>
-<pinref part="U2" gate="G$1" pin="GND"/>
 <pinref part="CN1" gate="G$1" pin="1"/>
+<pinref part="U2" gate="A" pin="GND"/>
+<junction x="93.98" y="83.82"/>
 </segment>
 <segment>
@@
 <pinref part="C11" gate="G$1" pin="+"/>
 <wire x1="71.12" y1="93.98" x2="71.12" y2="96.52" width="0.1524" layer="91"/>
-<wire x1="71.12" y1="96.52" x2="76.2" y2="96.52" width="0.1524" layer="91"/>
+<wire x1="71.12" y1="96.52" x2="78.74" y2="96.52" width="0.1524" layer="91"/>
 <pinref part="C10" gate="G$1" pin="1"/>
 <wire x1="60.96" y1="96.52" x2="71.12" y2="96.52" width="0.1524" layer="91"/>
@@
 <pinref part="D1" gate="G$1" pin="C"/>
 <junction x="60.96" y="96.52"/>
-<pinref part="U2" gate="G$1" pin="IN"/>
+<pinref part="U2" gate="A" pin="VIN"/>
 </segment>
 </net>
@@
 </segment>
 <segment>
-<wire x1="91.44" y1="96.52" x2="96.52" y2="96.52" width="0.1524" layer="91"/>
-<wire x1="96.52" y1="96.52" x2="99.06" y2="96.52" width="0.1524" layer="91"/>
-<wire x1="99.06" y1="96.52" x2="99.06" y2="104.14" width="0.1524" layer="91"/>
+<wire x1="149.86" y1="96.52" x2="152.4" y2="96.52" width="0.1524" layer="91"/>
+<wire x1="152.4" y1="96.52" x2="152.4" y2="104.14" width="0.1524" layer="91"/>
 <pinref part="C12" gate="G$1" pin="+"/>
-<wire x1="96.52" y1="93.98" x2="96.52" y2="96.52" width="0.1524" layer="91"/>
+<wire x1="149.86" y1="93.98" x2="149.86" y2="96.52" width="0.1524" layer="91"/>
 <pinref part="C13" gate="G$1" pin="1"/>
-<wire x1="99.06" y1="96.52" x2="106.68" y2="96.52" width="0.1524" layer="91"/>
-<wire x1="106.68" y1="96.52" x2="106.68" y2="93.98" width="0.1524" layer="91"/>
-<junction x="96.52" y="96.52"/>
-<junction x="99.06" y="96.52"/>
+<wire x1="152.4" y1="96.52" x2="160.02" y2="96.52" width="0.1524" layer="91"/>
+<wire x1="160.02" y1="96.52" x2="160.02" y2="93.98" width="0.1524" layer="91"/>
+<junction x="149.86" y="96.52"/>
+<junction x="152.4" y="96.52"/>
 <pinref part="SUPPLY2" gate="G$1" pin="1.8V"/>
-<pinref part="U2" gate="G$1" pin="OUT"/>
+<pinref part="U2" gate="A" pin="VOUT"/>
+<wire x1="149.86" y1="96.52" x2="109.22" y2="96.52" width="0.1524" layer="91"/>
 </segment>
 <segment>
@@
 <segment>
 <pinref part="F1" gate="G$1" pin="1"/>
-<wire x1="33.02" y1="96.52" x2="22.86" y2="96.52" width="0.1524" layer="91"/>
+<wire x1="33.02" y1="96.52" x2="27.94" y2="96.52" width="0.1524" layer="91"/>
 <label x="27.94" y="96.52" size="1.27" layer="95"/>
 <pinref part="CN1" gate="G$1" pin="2"/>
